Commit message: Turtle bot build completed

File: turtle_brick/urdf/turtle.urdf (robot description, URDF)
Before this commit: robot turtle_bot, 2 links, 1 joints
Links:
- added link pole; visual cylinder length=0.6 radius=0.05
- added link wheel; visual sphere radius=0.04
- link platform: geometry visual cylinder length=0.1 radius=0.7
Joints:
- added joint base_to_pole: type fixed, parent base_link, child pole, axis 0 0 1
- added joint wheel_to_base: type floating, parent base_link, child wheel
- joint base_to_platform: axis (none) -> 0 0 1; parent base_link -> pole; type fixed -> continuous

Commit message: Edited Robot urdf to touch the floor

File: turtle_brick/urdf/turtle.urdf (robot description, URDF)
Before this commit: robot turtle_bot, 4 links, 3 joints
Links:
- link pole: geometry visual cylinder length=1.4 radius=0.03
- link wheel: geometry visual sphere radius=0.09
Joints:
- joint wheel_to_base: origin (none) -> xyz=0 0 0.2 rpy=0 0 0

Commit message: Fine tuned urdf to match specifications

File: turtle_brick/urdf/turtle.urdf (robot description, URDF)
Before this commit: robot turtle_bot, 4 links, 3 joints
Links:
- added link stem; visual cylinder length=0.5 radius=0.02
- link pole: geometry visual cylinder length=1.1 radius=0.03
Joints:
- removed joint base_to_platform
- removed joint wheel_to_base
- added joint base_to_stem: type continuous, parent base_link, child stem, axis 0 0 1
- added joint pole_to_platform: type continuous, parent pole, child platform, axis 1 0 0
- added joint stem_to_wheel: type continuous, parent stem, child wheel, axis 1 0 0
- joint base_to_pole: axis 0 0 1 -> (none)
