Commit message: Attempt to load config yaml

File: turtle_brick/urdf/turtle.urdf.xacro (robot description, xacro)
@@ -1,4 +1,7 @@
 <?xml version="1.0"?>
-<robot name="turtle_bot">
+<robot xmlns:xacro="http://www.ros.org/wiki/xacro">
+<xacro:property name="yaml_file" value="$(find package)/turtle.yaml" />
+<xacro:property name="props" value="${xacro.load_yaml(yaml_file)['/**']['ros__parameters']}" />
+<xacro:property name="myprop"  value="${props['platform_height']}" />
   <link name="base_link">
     <visual>
@@ -14,5 +17,5 @@
   <link name="platform">
     <visual>
-      <origin xyz="0 0 1.5" rpy="0 0 0"/>
+      <origin xyz="0 0 ${myprop}" rpy="0 0 0"/>
       <geometry>
         <cylinder length="0.1" radius="0.7"/>

Commit message: create a show and run xml launch, customize urdf with xacro and yaml

File: turtle_brick/urdf/turtle.urdf.xacro (robot description, xacro)
@@ -1,7 +1,11 @@
 <?xml version="1.0"?>
-<robot xmlns:xacro="http://www.ros.org/wiki/xacro">
-<xacro:property name="yaml_file" value="$(find package)/turtle.yaml" />
+<robot name="turtle_bot" xmlns:xacro="http://www.ros.org/wiki/xacro">
+<!-- Get the path to the yaml file relative to the package -->
+<!-- config.yaml should have been installed in setup.py -->
+<xacro:property name="yaml_file" value="$(find turtle_brick)/turtle.yaml" />
+<!-- load values from yaml file which are stored in a dictionary called props-->
 <xacro:property name="props" value="${xacro.load_yaml(yaml_file)['/**']['ros__parameters']}" />
-<xacro:property name="myprop"  value="${props['platform_height']}" />
+<!-- access an individual variable -->
+<xacro:property name="platform_height"  value="${props['platform_height']}" />
   <link name="base_link">
     <visual>
@@ -17,7 +21,7 @@
   <link name="platform">
     <visual>
-      <origin xyz="0 0 ${myprop}" rpy="0 0 0"/>
+      <origin xyz="0 0 2" rpy="0 0 0"/>
       <geometry>
-        <cylinder length="0.1" radius="0.7"/>
+        <cylinder length="0.2" radius="0.7"/>
       </geometry>
       <material name="Red">
@@ -30,5 +34,5 @@
       <origin xyz="0 0 1" rpy="0 0 0"/>
       <geometry>
-        <cylinder length="1.1" radius="0.03"/>
+        <cylinder length="${platform_height}" radius="0.03"/>
       </geometry>
       <material name="Blue">
@@ -61,20 +65,24 @@
   <joint name="base_to_stem" type="continuous">
     <axis xyz="0 0 1" />
-      <parent link="base_link"/>
-      <child link="stem"/>
+    <origin xyz="0 0 0"/>
+    <parent link="base_link"/>
+    <child link="stem"/>
   </joint>
   <joint name="stem_to_wheel" type="continuous">
     <axis xyz="1 0 0" />
-      <parent link="stem"/>
-      <child link="wheel"/>
+    <origin xyz="0 0 0"/>
+    <parent link="stem"/>
+    <child link="wheel"/>
   </joint>
   <joint name="base_to_pole" type="fixed">
-      <parent link="base_link"/>
-      <child link="pole"/>
+    <origin xyz="0 0 0" />
+    <parent link="base_link"/>
+    <child link="pole"/>
   </joint>
   <joint name="pole_to_platform" type="continuous">
     <axis xyz="1 0 0" />
-      <parent link="pole"/>
-      <child link="platform"/>
+    <origin xyz="0 0 0"/>
+    <parent link="pole"/>
+    <child link="platform"/>
   </joint>
 </robot>

Commit message: Create xml launch files

File: turtle_brick/urdf/turtle.urdf.xacro (robot description, xacro)
@@ -8,4 +8,7 @@
 <!-- access an individual variable -->
 <xacro:property name="platform_height"  value="${props['platform_height']}" />
+<xacro:property name="wheel_radius"  value="${props['wheel_radius']}" />
+<!-- <xacro:property name="max_velocity"  value="${props['max_velocity']}" />
+<xacro:property name="gravity_accel"  value="${props['gravity_accel']}" /> -->
   <link name="base_link">
     <visual>
@@ -21,5 +24,5 @@
   <link name="platform">
     <visual>
-      <origin xyz="0 0 2" rpy="0 0 0"/>
+      <origin xyz="0 0 ${platform_height}" rpy="0 0 0"/>
       <geometry>
         <cylinder length="0.2" radius="0.7"/>
@@ -45,5 +48,5 @@
       <origin xyz="0 0 0" rpy="0 0 0"/>
         <geometry>
-          <sphere radius="0.09"/>
+          <sphere radius="${wheel_radius}"/>
         </geometry>
           <material name="Yellow">
@@ -63,5 +66,5 @@
     </visual>
   </link>
-  <joint name="base_to_stem" type="continuous">
+  <joint name="j1" type="continuous">
     <axis xyz="0 0 1" />
     <origin xyz="0 0 0"/>
@@ -69,9 +72,15 @@
     <child link="stem"/>
   </joint>
-  <joint name="stem_to_wheel" type="continuous">
+  <joint name="j2" type="continuous">
     <axis xyz="1 0 0" />
     <origin xyz="0 0 0"/>
     <parent link="stem"/>
     <child link="wheel"/>
+  </joint>
+  <joint name="j3" type="continuous">
+    <axis xyz="1 0 0" />
+    <origin xyz="0 0 0"/>
+    <parent link="pole"/>
+    <child link="platform"/>
   </joint>
   <joint name="base_to_pole" type="fixed">
@@ -80,9 +89,3 @@
     <child link="pole"/>
   </joint>
-  <joint name="pole_to_platform" type="continuous">
-    <axis xyz="1 0 0" />
-    <origin xyz="0 0 0"/>
-    <parent link="pole"/>
-    <child link="platform"/>
-  </joint>
 </robot>

Commit message: Robot moves toward goal pose

File: turtle_brick/urdf/turtle.urdf.xacro (robot description, xacro)
@@ -11,4 +11,5 @@
 <!-- <xacro:property name="max_velocity"  value="${props['max_velocity']}" />
 <xacro:property name="gravity_accel"  value="${props['gravity_accel']}" /> -->
+<!-- <xacro:property name="base_link_origin"  value="${}" /> -->
   <link name="base_link">
     <visual>
@@ -66,5 +67,5 @@
     </visual>
   </link>
-  <joint name="j1" type="continuous">
+  <joint name="j1" type="fixed">
     <axis xyz="0 0 1" />
     <origin xyz="0 0 0"/>
@@ -72,5 +73,5 @@
     <child link="stem"/>
   </joint>
-  <joint name="j2" type="continuous">
+  <joint name="j2" type="fixed">
     <axis xyz="1 0 0" />
     <origin xyz="0 0 0"/>
@@ -78,5 +79,5 @@
     <child link="wheel"/>
   </joint>
-  <joint name="j3" type="continuous">
+  <joint name="j3" type="fixed">
     <axis xyz="1 0 0" />
     <origin xyz="0 0 0"/>

Commit message: Robot catches the brick

File: turtle_brick/urdf/turtle.urdf.xacro (robot description, xacro)
@@ -16,5 +16,5 @@
       <origin xyz="0 0 0.5" rpy="0 0 0"/>
       <geometry>
-        <box size="0.5 0.5 0.5"/>
+        <box size="${platform_height / (platform_height*2)} ${platform_height / (platform_height*2)} ${platform_height / (platform_height*2)}"/>
       </geometry>
       <material name="White">
@@ -27,5 +27,5 @@
       <origin xyz="0 0 ${platform_height}" rpy="0 0 0"/>
       <geometry>
-        <cylinder length="0.2" radius="0.7"/>
+        <cylinder length="${platform_height/10}" radius="0.7"/>
       </geometry>
       <material name="Red">

Commit message: Catcher node completed, robot can determine if it can catch brick

File: turtle_brick/urdf/turtle.urdf.xacro (robot description, xacro)
@@ -1,15 +1,11 @@
-<?xml version="1.0"?>
 <robot name="turtle_bot" xmlns:xacro="http://www.ros.org/wiki/xacro">
-<!-- Get the path to the yaml file relative to the package -->
-<!-- config.yaml should have been installed in setup.py -->
-<xacro:property name="yaml_file" value="$(find turtle_brick)/turtle.yaml" />
-<!-- load values from yaml file which are stored in a dictionary called props-->
-<xacro:property name="props" value="${xacro.load_yaml(yaml_file)['/**']['ros__parameters']}" />
-<!-- access an individual variable -->
-<xacro:property name="platform_height"  value="${props['platform_height']}" />
-<xacro:property name="wheel_radius"  value="${props['wheel_radius']}" />
-<!-- <xacro:property name="max_velocity"  value="${props['max_velocity']}" />
-<xacro:property name="gravity_accel"  value="${props['gravity_accel']}" /> -->
-<!-- <xacro:property name="base_link_origin"  value="${}" /> -->
+  <!-- Get the path to the yaml file relative to the package -->
+  <!-- config.yaml should have been installed in setup.py -->
+  <xacro:property name="yaml_file" value="$(find turtle_brick)/turtle.yaml" />
+  <!-- load values from yaml file which are stored in a dictionary called props-->
+  <xacro:property name="props" value="${xacro.load_yaml(yaml_file)['/**']['ros__parameters']}" />
+  <!-- access an individual variable -->
+  <xacro:property name="platform_height"  value="${props['platform_height']}" />
+  <xacro:property name="wheel_radius"  value="${props['wheel_radius']}" />
   <link name="base_link">
     <visual>
@@ -68,23 +64,23 @@
   </link>
   <joint name="j1" type="fixed">
+    <!-- <origin xyz="0 0 -0.5"/> -->
     <axis xyz="0 0 1" />
-    <origin xyz="0 0 0"/>
     <parent link="base_link"/>
     <child link="stem"/>
   </joint>
   <joint name="j2" type="fixed">
+    <!-- <origin xyz="0 0 ${-(0.5 + wheel_radius)}"/> -->
     <axis xyz="1 0 0" />
-    <origin xyz="0 0 0"/>
     <parent link="stem"/>
     <child link="wheel"/>
   </joint>
   <joint name="j3" type="fixed">
+    <!-- <origin xyz="0 0 ${platform_height - platform_height/10}"/> -->
     <axis xyz="1 0 0" />
-    <origin xyz="0 0 0"/>
     <parent link="pole"/>
     <child link="platform"/>
   </joint>
   <joint name="base_to_pole" type="fixed">
-    <origin xyz="0 0 0" />
+    <!-- <origin xyz="0 0 0"/> -->
     <parent link="base_link"/>
     <child link="pole"/>
